File: _autosave-deneme.kicad_pcb (KiCad board)
At the start: 2 copper layers, 79 x 66.8 mm, 70 parts, among them J1 USB_C_Receptacle_USB2.0_16P, J2 Conn_01x04_Pin, J3 LORA_USART2_SOCKETS, J4 RJ45, SW1 SW_SPDT, U1 STM32F103C8T6, U2 AMS1117-3.3, U3 MAX485E, U4 ESDS302DBVR, U5 USBLC6-2SC6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

Commit message: added led resistors
Routing:
- net GND: track 50.0 -> 47.3 mm
Changed lines of the file:
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@@
 	)
 	(segment
-		(start 194.435 73.445)
-		(end 193.84 72.85)
-		(width 0.2)
-		(layer "F.Cu")
-		(net 1)
-	)
-	(segment
-		(start 202.07 77.82)
-		(end 202.45 77.44)
-		(width 0.2)
-		(layer "F.Cu")
-		(net 1)
-	)
-	(segment
 		(start 161.045 64.53)
 		(end 160.21 64.53)
@@
 	)
 	(segment
-		(start 200.77 77.82)
-		(end 202.07 77.82)
-		(width 0.2)
-		(layer "F.Cu")
-		(net 1)
-	)
-	(segment
 		(start 156.62 61.675)
 		(end 155.165 61.675)
@@
 	)
 	(segment
-		(start 185.695 72.5)
-		(end 198.13 60.065)
+		(start 203.225 77.825)
+		(end 203.225 76.125)
 		(width 0.5)
 		(layer "F.Cu")
@@
 	)
 	(segment
-		(start 203.225 77.825)
-		(end 203.225 76.125)
+		(start 185.695 72.5)
+		(end 198.13 60.065)
 		(width 0.5)
 		(layer "F.Cu")
@@
 	)
 	(segment
+		(start 195.81 79.12)
+		(end 201.93 79.12)
+		(width 0.5)
+		(layer "F.Cu")
+		(net 6)
+	)
+	(segment
 		(start 203 75.9)
 		(end 203.225 76.125)
@@
 	)
 	(segment
-		(start 195.62 78.93)
-		(end 202.12 78.93)
-		(width 0.5)
-		(layer "F.Cu")
-		(net 6)
-	)
-	(segment
 		(start 186.81 96.09)
 		(end 186.81 91.845)
@@
 	)
 	(segment
-		(start 202.12 78.93)
-		(end 203.225 77.825)
-		(width 0.5)
-		(layer "F.Cu")
-		(net 6)
-	)
-	(segment
 		(start 198.13 57.445)
 		(end 196.47 57.445)
@@
 	)
 	(segment
-		(start 195.62 78.93)
-		(end 192.665 75.975)
-		(width 0.5)
-		(layer "F.Cu")
-		(net 6)
-	)
-	(segment
 		(start 176.01 88.51)
 		(end 176.01 95.67)
@@
 	)
 	(segment
+		(start 201.93 79.12)
+		(end 203.225 77.825)
+		(width 0.5)
+		(layer "F.Cu")
+		(net 6)
+	)
+	(segment
 		(start 196.47 57.445)
 		(end 195.5 56.475)
@@
 		(width 0.5)
 		(layer "F.Cu")
+		(net 6)
+	)
+	(segment
+		(start 192.665 75.975)
+		(end 195.81 79.12)
+		(width 0.5)
+		(layer "F.Cu")
